File: circuit/auto-headlight-control-system/auto-headlight-control-system.sch (KiCad schematic (older format))
At the start: 16 parts, among them J1 Serial_Tx_1, J2 Serial_GND_1, J3 Serial_Tx_2, J4 Serial_GND_2, M1 SG90, T1 SN65HVD230, T2 SN65HVD230, U1 STM32_L, U2 STM32_R, U3 STM32_L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

Commit message: Add: gerber and Fix
Parts:
- R1: footprint Resistor_THT:R_Axial_DIN0207_L6.3mm_D2.5mm_P7.62mm_Horizontal -> Resistor_THT:R_Axial_DIN0207_L6.3mm_D2.5mm_P2.54mm_Vertical
Changed lines of the file:
@@
 3V3_1
 Wire Wire Line
-	2500 2650 2700 2650
-Wire Wire Line
 	2500 2750 2700 2750
 Wire Wire Line
@@
 	2350 4050 2550 4050
 Wire Wire Line
-	3750 3700 3900 3700
-Wire Wire Line
 	3750 3800 3900 3800
 Wire Wire Line
@@
 Wire Wire Line
 	3750 4650 3900 4650
-Wire Wire Line
-	3750 4750 3900 4750
 Wire Wire Line
 	3750 4850 3900 4850
@@
 F 0 "R1" H 5470 2546 50  0000 L CNN
 F 1 "100ohm" H 5470 2455 50  0000 L CNN
-F 2 "Resistor_THT:R_Axial_DIN0207_L6.3mm_D2.5mm_P7.62mm_Horizontal" V 5330 2500 50  0001 C CNN
+F 2 "Resistor_THT:R_Axial_DIN0207_L6.3mm_D2.5mm_P2.54mm_Vertical" V 5330 2500 50  0001 C CNN
 F 3 "~" H 5400 2500 50  0001 C CNN
 	1    5400 2500
@@
 	1    0    0    -1
 $EndComp
+Wire Wire Line
+	3750 4750 3900 4750
+Wire Wire Line
+	2500 2650 2700 2650
+Wire Wire Line
+	3750 3700 3900 3700
 $EndSCHEMATC
